Commit message: .xacro with rtb map
urdf

File: src/my_robot/urdf/my_robot.xacro (robot description, xacro)
@@ -144,4 +144,14 @@
     </visual>
  </link>
+ <link name='camera_link_optical'>
+ </link>
+  <joint type="fixed" name="camera_optical_joint">
+    <origin xyz="0 0 0" rpy="-1.5707 0 -1.5707"/>
+    <parent link="camera"/>
+    <child link="camera_link_optical"/>
+    <axis xyz="0 1 0" rpy="0 0 0"/>
+    <limit effort="10000" velocity="1000"/>
+    <dynamics damping="1.0" friction="1.0"/>
+  </joint>
   <joint type="fixed" name="camera_joint">
     <origin xyz="0.2 0 0" rpy="0 0 0"/>
